File: can-ortholinear-keyboard.sch (KiCad schematic (older format))
At the start: 173 parts, among them SW1 SW_Push, SW10 SW_Push, SW11 SW_Push, SW12 SW_Push, SW13 SW_Push, SW14 SW_Push, SW15 SW_Push, SW16 SW_Push, SW17 SW_Push, SW18 SW_Push, SW19 SW_Push, SW2 SW_Push, SW20 SW_Push, SW21 SW_Push, SW22 SW_Push, SW23 SW_Push, SW24 SW_Push, SW25 SW_Push, SW26 SW_Push, SW27 SW_Push, SW28 SW_Push, SW29 SW_Push, SW3 SW_Push, SW30 SW_Push, SW31 SW_Push, SW32 SW_Push, SW33 SW_Push, SW34 SW_Push, SW35 SW_Push, SW36 SW_Push, SW37 SW_Push, SW38 SW_Push, SW39 SW_Push, SW4 SW_Push, SW40 SW_Push, SW41 SW_Push, SW42 SW_Push, SW43 SW_Push, SW44 SW_Push, SW45 SW_Push, SW46 SW_Push, SW47 SW_Push, SW48 SW_Push, SW49 SW_Push, SW5 SW_Push, SW50 SW_Push, SW51 SW_Push, SW52 SW_Push, SW53 SW_Push, SW54 SW_Push, SW55 SW_Push, SW56 SW_Push, SW57 SW_Push, SW58 SW_Push, SW59 SW_Push, SW6 SW_Push, SW60 SW_Push, SW61 SW_Push, SW62 SW_Push, SW63 SW_Push, SW64 SW_Push, SW65 SW_Push, SW66 SW_Push, SW67 SW_Push, SW68 SW_Push, SW69 SW_Push, SW7 SW_Push, SW70 SW_Push, SW71 SW_Push, SW72 SW_Push, SW73 SW_Push, SW74 SW_Push, SW75 SW_Push, SW76 SW_Push, SW77 SW_SPST, SW78 SW_Push, SW79 SW_Push, SW8 SW_Push, SW80 SW_Push, SW81 SW_Push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

Commit message: Assign footprints except 2 toggle switches.
Parts:
- SW1, SW10, SW11, SW12, SW13, SW14, SW15, SW16, SW17, SW18, SW19, SW2, SW20, SW21, SW22, SW23, SW24, SW25, SW26, SW27, SW28, SW29, SW3, SW31, SW32, SW33, SW34, SW35, SW36, SW37, SW38, SW39, SW4, SW40, SW42, SW43, SW44, SW45, SW46, SW47, SW48, SW49, SW5, SW50, SW51, SW52, SW53, SW54, SW55, SW56, SW57, SW58, SW59, SW6, SW60, SW61, SW62, SW63, SW64, SW65, SW66, SW67, SW68, SW69, SW7, SW70, SW71, SW72, SW74, SW75, SW76, SW79, SW8, SW80, SW81, SW83, SW84, SW85, SW86, SW9: footprint (none) -> Button_Switch_Keyboard:SW_Cherry_MX_1.00u_PCB
- SW30, SW41, SW73, SW78: footprint (none) -> Button_Switch_Keyboard:SW_Cherry_MX_2.00u_PCB

Commit message: Placed every component on PCB.
Parts:
- SW73: footprint Button_Switch_Keyboard:SW_Cherry_MX_2.00u_PCB -> Button_Switch_Keyboard:SW_Cherry_MX_1.00u_PCB
- SW74: footprint Button_Switch_Keyboard:SW_Cherry_MX_1.00u_PCB -> Button_Switch_Keyboard:SW_Cherry_MX_2.00u_PCB
- SW77, SW82: footprint (none) -> Connector_PinSocket_2.54mm:PinSocket_1x02_P2.54mm_Vertical
Connections:
- net Row2: now also D79.1 (K)
- net Row3: no longer D79.1 (K)
Other:
- moved on the sheet: D79, SW79
Changed lines of the file:
@@
 F 0 "SW73" H 12750 3735 50  0000 C CNN
 F 1 "SW_Push" H 12750 3644 50  0000 C CNN
-F 2 "Button_Switch_Keyboard:SW_Cherry_MX_2.00u_PCB" H 12750 3650 50  0001 C CNN
+F 2 "Button_Switch_Keyboard:SW_Cherry_MX_1.00u_PCB" H 12750 3650 50  0001 C CNN
 F 3 "~" H 12750 3650 50  0001 C CNN
 	1    12750 3450
@@
 F 0 "SW74" H 12750 4485 50  0000 C CNN
 F 1 "SW_Push" H 12750 4394 50  0000 C CNN
-F 2 "Button_Switch_Keyboard:SW_Cherry_MX_1.00u_PCB" H 12750 4400 50  0001 C CNN
+F 2 "Button_Switch_Keyboard:SW_Cherry_MX_2.00u_PCB" H 12750 4400 50  0001 C CNN
 F 3 "~" H 12750 4400 50  0001 C CNN
 	1    12750 4200
@@
 L Switch:SW_Push SW79
 U 1 1 5F0DE7F6
-P 13600 4200
-F 0 "SW79" H 13600 4485 50  0000 C CNN
-F 1 "SW_Push" H 13600 4394 50  0000 C CNN
-F 2 "Button_Switch_Keyboard:SW_Cherry_MX_1.00u_PCB" H 13600 4400 50  0001 C CNN
-F 3 "~" H 13600 4400 50  0001 C CNN
-	1    13600 4200
+P 13600 3450
+F 0 "SW79" H 13600 3735 50  0000 C CNN
+F 1 "SW_Push" H 13600 3644 50  0000 C CNN
+F 2 "Button_Switch_Keyboard:SW_Cherry_MX_1.00u_PCB" H 13600 3650 50  0001 C CNN
+F 3 "~" H 13600 3650 50  0001 C CNN
+	1    13600 3450
 	1    0    0    -1
 $EndComp
@@
 L Diode:1N4148 D79
 U 1 1 5F0DE800
-P 13800 4350
-F 0 "D79" V 13846 4270 50  0000 R CNN
-F 1 "1N4148" V 13755 4270 50  0000 R CNN
-F 2 "Diode_THT:D_DO-35_SOD27_P7.62mm_Horizontal" H 13800 4175 50  0001 C CNN
-F 3 "https://assets.nexperia.com/documents/data-sheet/1N4148_1N4448.pdf" H 13800 4350 50  0001 C CNN
-	1    13800 4350
+P 13800 3600
+F 0 "D79" V 13846 3520 50  0000 R CNN
+F 1 "1N4148" V 13755 3520 50  0000 R CNN
+F 2 "Diode_THT:D_DO-35_SOD27_P7.62mm_Horizontal" H 13800 3425 50  0001 C CNN
+F 3 "https://assets.nexperia.com/documents/data-sheet/1N4148_1N4448.pdf" H 13800 3600 50  0001 C CNN
+	1    13800 3600
 	0    -1   -1   0
 $EndComp
@@
 Wire Wire Line
 	12950 3750 12100 3750
-Wire Wire Line
-	14650 4500 13800 4500
 Connection ~ 2750 4500
 Wire Wire Line
@@
 Wire Wire Line
 	12950 4500 12100 4500
-Connection ~ 13800 4500
-Wire Wire Line
-	13800 4500 12950 4500
 Wire Wire Line
 	14650 5250 13800 5250
@@
 	13400 5700 13400 4950
 Connection ~ 13400 2700
-Connection ~ 13400 4200
 Connection ~ 13400 4950
-Wire Wire Line
-	13400 4950 13400 4200
 Wire Wire Line
 	12550 5700 12550 4950
@@
 F 0 "SW82" H 14450 2185 50  0000 C CNN
 F 1 "SW_SPST" H 14450 2094 50  0000 C CNN
-F 2 "" H 14450 1950 50  0001 C CNN
+F 2 "Connector_PinSocket_2.54mm:PinSocket_1x02_P2.54mm_Vertical" H 14450 1950 50  0001 C CNN
 F 3 "~" H 14450 1950 50  0001 C CNN
 	1    14450 1950
@@
 F 0 "SW77" H 13600 2185 50  0000 C CNN
 F 1 "SW_SPST" H 13600 2094 50  0000 C CNN
-F 2 "" H 13600 1950 50  0001 C CNN
+F 2 "Connector_PinSocket_2.54mm:PinSocket_1x02_P2.54mm_Vertical" H 13600 1950 50  0001 C CNN
 F 3 "~" H 13600 1950 50  0001 C CNN
 	1    13600 1950
@@
 	14250 1950 14250 3450
 Wire Wire Line
-	13400 2700 13400 4200
-Wire Wire Line
-	12950 3750 14650 3750
+	13400 2700 13400 3450
+Wire Wire Line
+	12950 3750 13800 3750
 Wire Wire Line
 	6150 6000 7850 6000
@@
 NoConn ~ 3000 8550
 NoConn ~ 3000 8850
+Connection ~ 13400 3450
+Connection ~ 13800 3750
+Wire Wire Line
+	13800 3750 14650 3750
+Wire Wire Line
+	12950 4500 14650 4500
+Wire Wire Line
+	13400 3450 13400 4950
 $EndSCHEMATC
