File: can-ortholinear-keyboard.kicad_pcb (KiCad board)
At the start: 2 copper layers, 289.6 x 115.8 mm, 173 parts, among them SW1 SW_Push, SW10 SW_Push, SW11 SW_Push, SW12 SW_Push, SW13 SW_Push, SW14 SW_Push, SW15 SW_Push, SW16 SW_Push, SW17 SW_Push, SW18 SW_Push, SW19 SW_Push, SW2 SW_Push, SW20 SW_Push, SW21 SW_Push, SW22 SW_Push, SW23 SW_Push, SW24 SW_Push, SW25 SW_Push, SW26 SW_Push, SW27 SW_Push, SW28 SW_Push, SW29 SW_Push, SW3 SW_Push, SW30 SW_Push, SW31 SW_Push, SW32 SW_Push, SW33 SW_Push, SW34 SW_Push, SW35 SW_Push, SW36 SW_Push, SW37 SW_Push, SW38 SW_Push, SW39 SW_Push, SW4 SW_Push, SW40 SW_Push, SW41 SW_Push, SW42 SW_Push, SW43 SW_Push, SW44 SW_Push, SW45 SW_Push, SW46 SW_Push, SW47 SW_Push, SW48 SW_Push, SW49 SW_Push, SW5 SW_Push, SW50 SW_Push, SW51 SW_Push, SW52 SW_Push, SW53 SW_Push, SW54 SW_Push, SW55 SW_Push, SW56 SW_Push, SW57 SW_Push, SW58 SW_Push, SW59 SW_Push, SW6 SW_Push, SW60 SW_Push, SW61 SW_Push, SW62 SW_Push, SW63 SW_Push, SW64 SW_Push, SW65 SW_Push, SW66 SW_Push, SW67 SW_Push, SW68 SW_Push, SW69 SW_Push, SW7 SW_Push, SW70 SW_Push, SW71 SW_Push, SW72 SW_Push, SW73 SW_Push, SW74 SW_Push, SW75 SW_Push, SW76 SW_Push, SW77 SW_SPST, SW78 SW_Push, SW79 SW_Push, SW8 SW_Push, SW80 SW_Push, SW81 SW_Push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

Commit message: Drew all the tracks.
Parts:
- moved D42 7.11 mm to (161.0, 50.8), turned to 0 degrees
- moved D43 7.11 mm to (161.0, 70.1), turned to 0 degrees
- moved D77 7.11 mm to (276.9, 50.8), turned to 0 degrees
Routing:
- net /Row5: track 0.00 -> 359.8 mm
- net /Row4: track 0.00 -> 331.0 mm
- net /Row3: track 0.00 -> 313.9 mm
- net /Row2: track 0.00 -> 301.3 mm
- net /Row1: track 0.00 -> 300.0 mm
- net /Row0: track 0.00 -> 258.1 mm
- net /Col14: track 0.00 -> 248.0 mm
- net /Col13: track 0.00 -> 225.4 mm
- net /Col0: track 0.00 -> 223.6 mm
- net /Col12: track 0.00 -> 213.9 mm
- net /Col1: track 0.00 -> 202.9 mm
- net /Col3: track 0.00 -> 189.7 mm
- net /Col11: track 0.00 -> 187.4 mm
- net /Col2: track 0.00 -> 186.6 mm
- net /Col10: track 0.00 -> 170.0 mm
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
Commit message: Silkscreen modifications.
Other:
- board text added: "Can Ortholinear Keyboard Rev. 0"
- board text added: "github.com/canaknesil/can-ortholinear-keyboard"

Commit message: Rerouted with thicker tracks.
Routing:
- net /Row3: track 313.9 -> 334.3 mm
- net /Col3: track 189.7 -> 169.6 mm
- net Net-(D43-Pad2): track 18.2 -> 29.9 mm
- net /Col13: track 225.4 -> 230.0 mm
- net Net-(D42-Pad2): track 19.2 -> 23.6 mm
- net /Col9: track 149.3 -> 153.5 mm
- net /Col0: track 223.6 -> 227.7 mm
- net /Col14: track 248.0 -> 252.0 mm
- net Net-(D55-Pad2): track 6.26 -> 9.31 mm
- net /Col8: track 130.3 -> 132.9 mm
- net /Row5: track 359.8 -> 357.6 mm
- net /Col2: track 186.6 -> 188.6 mm
- net /Col4: track 152.2 -> 150.5 mm
- net Net-(D5-Pad2): track 12.3 -> 13.2 mm
- net Net-(D2-Pad2): track 12.3 -> 13.2 mm
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Other:
- net class Default: clearance 0.2 -> 0.25; trace_width 0.25 -> 0.5
- rule trace_clearance: 0.2 -> 0.25
- rule trace_min: 0.2 -> 0.4

Commit message: Removed the gap between switches and rerouted.
Parts:
- moved SW86 3.78 mm to (318.0, 131.3)
- moved SW85 3.70 mm to (318.0, 112.3)
- moved SW84 3.64 mm to (318.0, 93.2)
- moved SW83 3.59 mm to (318.0, 74.2)
- moved D78 3.58 mm to (302.3, 69.7)
- moved SW81 3.54 mm to (299.0, 131.3)
- moved SW80 3.45 mm to (299.0, 112.3)
- moved SW78 3.44 mm to (308.5, 55.1)
- moved D84 3.43 mm to (305.9, 103.3)
- moved D85 3.43 mm to (305.9, 122.3)
- moved D83 3.43 mm to (305.9, 83.8)
- moved SW79 3.34 mm to (299.0, 74.2)
- moved SW76 3.30 mm to (279.9, 131.3)
- moved SW74 3.27 mm to (289.4, 93.2)
- moved SW75 3.21 mm to (279.9, 112.3)
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Routing:
- net /Row3: track 334.3 -> 310.5 mm
- net /Row2: track 301.2 -> 296.5 mm
- net /Col13: track 230.0 -> 225.7 mm
- net /Col0: track 227.7 -> 223.6 mm
- net /Row4: track 330.6 -> 327.0 mm
- net /Col14: track 252.0 -> 248.4 mm
- net Net-(D55-Pad2): track 9.31 -> 5.87 mm
- net /Col9: track 153.5 -> 150.2 mm
- net /Col1: track 203.8 -> 200.8 mm
- net /Col2: track 188.6 -> 185.7 mm
- net /Col8: track 132.9 -> 130.2 mm
- net /Col12: track 214.6 -> 212.2 mm
- net /Col11: track 187.5 -> 185.2 mm
- net /Col3: track 169.6 -> 167.4 mm
- net /Col10: track 170.0 -> 167.9 mm
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Other:
- board size 289.6 x 115.8 mm -> 285.8 x 114.4 mm
